Commit message: fix(viz): correct transforms and clock sync for RViz/Gazebo
- Fix 'blob' car in RViz by renaming URDF joints to match Gazebo SDF (steering_joint -> wheel_steering_joint).
- Fix missing wheel TFs by explicitly listing joints in SDF JointStatePublisher plugin.
- Fix 'no car' issue by restoring correct 'saye/' frame prefix in launch and bridge.
- Fix RViz timestamp errors by enforcing 'use_sim_time=True' in launch and absolute '/clock' topic in bridge.
- Comment out saye_localization dependency in launch file to fix build error.
- Verified compatibility with Gazebo Harmonic and ROS 2 Jazzy.

File: saye_description/urdf/saye.urdf (robot description, URDF)
Before this commit: robot saye, 7 links, 6 joints
Joints:
- removed joint front_left_steering_joint
- removed joint front_right_steering_joint
- added joint front_left_wheel_steering_joint: type continuous, parent base_link, child front_left_wheel_steering_link, origin xyz=0.112 0.10 0 rpy=0 0 0, axis 0 0 1
- added joint front_right_wheel_steering_joint: type continuous, parent base_link, child front_right_wheel_steering_link, origin xyz=0.112 -0.10 0 rpy=0 0 0, axis 0 0 1

Commit message: fix(saye_model): correct physics, inertia and sensor config
- Corrected wheel inertia tensors (swapped ixx/iyy)
- Added kp/kd stiffness to wheels for stability
- Reduced max acceleration to prevent pitching
- Fixed SDF syntax error in base_link sensors
- Increased Odom and JointState update rates to 100Hz for smoother TF

File: saye_description/urdf/saye.urdf (robot description, URDF)
Before this commit: robot saye, 7 links, 6 joints
Links:
- added link lidar_link
Joints:
- added joint lidar_joint: type fixed, parent base_link, child lidar_link, origin xyz=0.05 0 0.12 rpy=0 0 0
